Commit message: incorpora ficha suministrada de los doce MG996R

File: Experimentos/modelos_gemelo_generados/realistic_provisional/nova_gazebo.urdf (robot description, URDF)
Before this commit: robot nova_sm3, 18 links, 17 joints
Joints:
- joint front_left_coxa_joint: limit lower=-0.60 upper=0.60 effort=0.7279245081300812 velocity=6.399540590645874 -> lower=-0.60 upper=0.60 effort=0.6838078712737128 velocity=6.368920779207378
- joint front_left_femur_joint: limit lower=-1.20 upper=1.20 effort=0.7279245081300812 velocity=6.399540590645874 -> lower=-1.20 upper=1.20 effort=0.6838078712737128 velocity=6.368920779207378
- joint front_left_tibia_joint: limit lower=-2.20 upper=0.10 effort=0.7279245081300812 velocity=6.399540590645874 -> lower=-2.20 upper=0.10 effort=0.6838078712737128 velocity=6.368920779207378
- joint front_right_coxa_joint: limit lower=-0.60 upper=0.60 effort=0.7279245081300812 velocity=6.399540590645874 -> lower=-0.60 upper=0.60 effort=0.6838078712737128 velocity=6.368920779207378
- joint front_right_femur_joint: limit lower=-1.20 upper=1.20 effort=0.7279245081300812 velocity=6.399540590645874 -> lower=-1.20 upper=1.20 effort=0.6838078712737128 velocity=6.368920779207378
- joint front_right_tibia_joint: limit lower=-2.20 upper=0.10 effort=0.7279245081300812 velocity=6.399540590645874 -> lower=-2.20 upper=0.10 effort=0.6838078712737128 velocity=6.368920779207378
- joint rear_left_coxa_joint: limit lower=-0.60 upper=0.60 effort=0.7279245081300812 velocity=6.399540590645874 -> lower=-0.60 upper=0.60 effort=0.6838078712737128 velocity=6.368920779207378
- joint rear_left_femur_joint: limit lower=-1.20 upper=1.20 effort=0.7279245081300812 velocity=6.399540590645874 -> lower=-1.20 upper=1.20 effort=0.6838078712737128 velocity=6.368920779207378
- joint rear_left_tibia_joint: limit lower=-2.20 upper=0.10 effort=0.7279245081300812 velocity=6.399540590645874 -> lower=-2.20 upper=0.10 effort=0.6838078712737128 velocity=6.368920779207378
- joint rear_right_coxa_joint: limit lower=-0.60 upper=0.60 effort=0.7279245081300812 velocity=6.399540590645874 -> lower=-0.60 upper=0.60 effort=0.6838078712737128 velocity=6.368920779207378
- joint rear_right_femur_joint: limit lower=-1.20 upper=1.20 effort=0.7279245081300812 velocity=6.399540590645874 -> lower=-1.20 upper=1.20 effort=0.6838078712737128 velocity=6.368920779207378
- joint rear_right_tibia_joint: limit lower=-2.20 upper=0.10 effort=0.7279245081300812 velocity=6.399540590645874 -> lower=-2.20 upper=0.10 effort=0.6838078712737128 velocity=6.368920779207378
