Commit message: crea perfiles fisicos emparejados para simuladores

File: src/nova_sm3_description/urdf/nova_sm3.ros2_control.xacro (robot description, xacro)
@@ -1,5 +1,5 @@
 <?xml version="1.0"?>
 <robot xmlns:xacro="http://www.ros.org/wiki/xacro">
-  <xacro:macro name="nova_ros2_control" params="use_fake_hardware:=true use_mujoco:=false use_gazebo:=false headless:=false">
+  <xacro:macro name="nova_ros2_control" params="use_fake_hardware:=true use_mujoco:=false use_gazebo:=false headless:=false mujoco_model:=''">
     <ros2_control name="NovaSM3System" type="system">
       <hardware>
@@ -10,5 +10,5 @@
         <xacro:if value="${use_mujoco}">
           <plugin>mujoco_ros2_control/MujocoSystemInterface</plugin>
-          <param name="mujoco_model">$(find nova_sm3_description)/mujoco/nova_sm3.xml</param>
+          <param name="mujoco_model">${mujoco_model}</param>
           <param name="headless">${headless}</param>
           <param name="sim_speed_factor">1.0</param>

File: src/nova_sm3_description/urdf/nova_sm3.urdf.xacro (robot description, xacro)
@@ -6,4 +6,12 @@
   <xacro:arg name="headless" default="false"/>
   <xacro:arg name="include_ros2_control" default="true"/>
+  <!-- Experimental scales shared with generated MuJoCo profiles. -->
+  <xacro:arg name="mass_scale" default="1.0"/>
+  <xacro:arg name="inertia_scale" default="1.0"/>
+  <xacro:arg name="joint_damping" default="0.08"/>
+  <xacro:arg name="joint_friction" default="0.03"/>
+  <xacro:arg name="actuator_effort" default="1.0787315"/>
+  <xacro:arg name="actuator_velocity" default="6.981317"/>
+  <xacro:arg name="mujoco_model" default="$(find nova_sm3_description)/mujoco/nova_sm3.xml"/>
   <xacro:include filename="$(find nova_sm3_description)/urdf/nova_sm3.materials.xacro"/>
   <xacro:include filename="$(find nova_sm3_description)/urdf/nova_sm3.ros2_control.xacro"/>
@@ -26,16 +34,22 @@
   <xacro:property name="body_height" value="0.075"/>
   <!-- Estimated distribution sums to the published approximate total 2.72 kg. -->
-  <xacro:property name="body_mass" value="1.20"/>
-  <xacro:property name="coxa_mass" value="0.12"/>
-  <xacro:property name="femur_mass" value="0.12"/>
-  <xacro:property name="tibia_mass" value="0.11"/>
-  <xacro:property name="foot_mass" value="0.03"/>
+  <xacro:property name="mass_scale" value="$(arg mass_scale)"/>
+  <xacro:property name="inertia_scale" value="$(arg inertia_scale)"/>
+  <xacro:property name="joint_damping" value="$(arg joint_damping)"/>
+  <xacro:property name="joint_friction" value="$(arg joint_friction)"/>
+  <xacro:property name="actuator_effort" value="$(arg actuator_effort)"/>
+  <xacro:property name="actuator_velocity" value="$(arg actuator_velocity)"/>
+  <xacro:property name="body_mass" value="${1.20*mass_scale}"/>
+  <xacro:property name="coxa_mass" value="${0.12*mass_scale}"/>
+  <xacro:property name="femur_mass" value="${0.12*mass_scale}"/>
+  <xacro:property name="tibia_mass" value="${0.11*mass_scale}"/>
+  <xacro:property name="foot_mass" value="${0.03*mass_scale}"/>
   <xacro:macro name="box_inertial" params="mass x y z origin_x:=0 origin_y:=0 origin_z:=0">
     <inertial>
       <origin xyz="${origin_x} ${origin_y} ${origin_z}"/>
       <mass value="${mass}"/>
-      <inertia ixx="${mass*(y*y+z*z)/12}" ixy="0" ixz="0"
-               iyy="${mass*(x*x+z*z)/12}" iyz="0"
-               izz="${mass*(x*x+y*y)/12}"/>
+      <inertia ixx="${inertia_scale*mass*(y*y+z*z)/12}" ixy="0" ixz="0"
+               iyy="${inertia_scale*mass*(x*x+z*z)/12}" iyz="0"
+               izz="${inertia_scale*mass*(x*x+y*y)/12}"/>
     </inertial>
   </xacro:macro>
@@ -50,6 +64,6 @@
       <origin xyz="${x} ${y} 0"/><axis xyz="${side} 0 0"/>
       <!-- Placeholder mechanical envelope; replace after physical calibration. -->
-      <limit lower="-0.60" upper="0.60" effort="1.0787315" velocity="6.981317"/>
-      <dynamics damping="0.08" friction="0.03"/>
+      <limit lower="-0.60" upper="0.60" effort="${actuator_effort}" velocity="${actuator_velocity}"/>
+      <dynamics damping="${joint_damping}" friction="${joint_friction}"/>
     </joint>
     <link name="${prefix}_femur_link">
@@ -61,6 +75,6 @@
       <parent link="${prefix}_coxa_link"/><child link="${prefix}_femur_link"/>
       <origin xyz="0 ${side*coxa_length} 0"/><axis xyz="0 1 0"/>
-      <limit lower="-1.20" upper="1.20" effort="1.0787315" velocity="6.981317"/>
-      <dynamics damping="0.08" friction="0.03"/>
+      <limit lower="-1.20" upper="1.20" effort="${actuator_effort}" velocity="${actuator_velocity}"/>
+      <dynamics damping="${joint_damping}" friction="${joint_friction}"/>
     </joint>
     <link name="${prefix}_tibia_link">
@@ -72,11 +86,11 @@
       <parent link="${prefix}_femur_link"/><child link="${prefix}_tibia_link"/>
       <origin xyz="0 0 ${-femur_length}"/><axis xyz="0 1 0"/>
-      <limit lower="-2.20" upper="0.10" effort="1.0787315" velocity="6.981317"/>
-      <dynamics damping="0.08" friction="0.03"/>
+      <limit lower="-2.20" upper="0.10" effort="${actuator_effort}" velocity="${actuator_velocity}"/>
+      <dynamics damping="${joint_damping}" friction="${joint_friction}"/>
     </joint>
     <link name="${prefix}_foot_link">
       <visual><geometry><sphere radius="0.018"/></geometry><material name="nova_grey"/></visual>
       <collision name="${prefix}_foot_collision"><geometry><sphere radius="0.018"/></geometry></collision>
-      <inertial><mass value="${foot_mass}"/><inertia ixx="0.0000039" ixy="0" ixz="0" iyy="0.0000039" iyz="0" izz="0.0000039"/></inertial>
+      <inertial><mass value="${foot_mass}"/><inertia ixx="${0.0000039*mass_scale*inertia_scale}" ixy="0" ixz="0" iyy="${0.0000039*mass_scale*inertia_scale}" iyz="0" izz="${0.0000039*mass_scale*inertia_scale}"/></inertial>
     </link>
     <joint name="${prefix}_foot_joint" type="fixed">
@@ -123,5 +137,5 @@
   <xacro:nova_leg prefix="rear_right"  x="${-hip_spacing_x/2}" y="${-hip_spacing_y/2}" side="-1"/>
   <xacro:if value="$(arg include_ros2_control)">
-    <xacro:nova_ros2_control use_fake_hardware="$(arg use_fake_hardware)" use_mujoco="$(arg use_mujoco)" use_gazebo="$(arg use_gazebo)" headless="$(arg headless)"/>
+    <xacro:nova_ros2_control use_fake_hardware="$(arg use_fake_hardware)" use_mujoco="$(arg use_mujoco)" use_gazebo="$(arg use_gazebo)" headless="$(arg headless)" mujoco_model="$(arg mujoco_model)"/>
   </xacro:if>
   <xacro:if value="$(arg use_gazebo)">

Commit message: depura campañas aisladas de MuJoCo

File: src/nova_sm3_description/urdf/nova_sm3.ros2_control.xacro (robot description, xacro)
@@ -1,5 +1,5 @@
 <?xml version="1.0"?>
 <robot xmlns:xacro="http://www.ros.org/wiki/xacro">
-  <xacro:macro name="nova_ros2_control" params="use_fake_hardware:=true use_mujoco:=false use_gazebo:=false headless:=false mujoco_model:=''">
+  <xacro:macro name="nova_ros2_control" params="use_fake_hardware:=true use_mujoco:=false use_gazebo:=false headless:=false mujoco_model:='' sim_speed_factor:=1.0">
     <ros2_control name="NovaSM3System" type="system">
       <hardware>
@@ -12,5 +12,5 @@
           <param name="mujoco_model">${mujoco_model}</param>
           <param name="headless">${headless}</param>
-          <param name="sim_speed_factor">1.0</param>
+          <param name="sim_speed_factor">${sim_speed_factor}</param>
         </xacro:if>
         <xacro:if value="${use_gazebo}">

File: src/nova_sm3_description/urdf/nova_sm3.urdf.xacro (robot description, xacro)
@@ -5,4 +5,5 @@
   <xacro:arg name="use_gazebo" default="false"/>
   <xacro:arg name="headless" default="false"/>
+  <xacro:arg name="sim_speed_factor" default="1.0"/>
   <xacro:arg name="include_ros2_control" default="true"/>
   <!-- Experimental scales shared with generated MuJoCo profiles. -->
@@ -137,5 +138,5 @@
   <xacro:nova_leg prefix="rear_right"  x="${-hip_spacing_x/2}" y="${-hip_spacing_y/2}" side="-1"/>
   <xacro:if value="$(arg include_ros2_control)">
-    <xacro:nova_ros2_control use_fake_hardware="$(arg use_fake_hardware)" use_mujoco="$(arg use_mujoco)" use_gazebo="$(arg use_gazebo)" headless="$(arg headless)" mujoco_model="$(arg mujoco_model)"/>
+    <xacro:nova_ros2_control use_fake_hardware="$(arg use_fake_hardware)" use_mujoco="$(arg use_mujoco)" use_gazebo="$(arg use_gazebo)" headless="$(arg headless)" mujoco_model="$(arg mujoco_model)" sim_speed_factor="$(arg sim_speed_factor)"/>
   </xacro:if>
   <xacro:if value="$(arg use_gazebo)">
